Commit message: add Manipulability & change urdf files to get joint_info

File: unitree_pybullet/unitree_pybullet/data/_a1/urdf/a1.urdf (robot description, URDF)
Before this commit: robot a1_description, 22 links, 21 joints
Links:
- removed link FL_lower
- removed link FL_toe
- removed link FL_upper
- removed link FL_upper_shoulder
- removed link FR_lower
- removed link FR_toe
- removed link FR_upper
- removed link FR_upper_shoulder
- removed link RL_lower
- removed link RL_toe
- removed link RL_upper
- removed link RL_upper_shoulder
- removed link RR_lower
- removed link RR_toe
- removed link RR_upper
- removed link RR_upper_shoulder
- added link FL_calf, mass 0.166; collision box size=0.2 0.016 0.016; visual mesh filename=../meshes/calf.stl scale=1 1 1
- added link FL_foot, mass 0.06; collision sphere radius=0.02; visual sphere radius=0.01
- added link FL_thigh, mass 1.013; collision box size=0.2 0.0245 0.034; visual mesh filename=../meshes/thigh.stl scale=1 1 1
- added link FR_calf, mass 0.166; collision box size=0.2 0.016 0.016; visual mesh filename=../meshes/calf.stl scale=1 1 1
- added link FR_foot, mass 0.06; collision sphere radius=0.02; visual sphere radius=0.01
- added link FR_thigh, mass 1.013; collision box size=0.2 0.0245 0.034; visual mesh filename=../meshes/thigh_mirror.stl scale=1 1 1
- added link RL_calf, mass 0.166; collision box size=0.2 0.016 0.016; visual mesh filename=../meshes/calf.stl scale=1 1 1
- added link RL_foot, mass 0.06; collision sphere radius=0.02; visual sphere radius=0.01
- added link RL_thigh, mass 1.013; collision box size=0.2 0.0245 0.034; visual mesh filename=../meshes/thigh.stl scale=1 1 1
- added link RR_calf, mass 0.166; collision box size=0.2 0.016 0.016; visual mesh filename=../meshes/calf.stl scale=1 1 1
- added link RR_foot, mass 0.06; collision sphere radius=0.02; visual sphere radius=0.01
- added link RR_thigh, mass 1.013; collision box size=0.2 0.0245 0.034; visual mesh filename=../meshes/thigh_mirror.stl scale=1 1 1
- added link base; visual box size=0.001 0.001 0.001
- link FL_hip: geometry collision cylinder length=0.04 radius=0.046; visual mesh filename=../meshes/hip.stl scale=1 1 1
- link FR_hip: geometry collision cylinder length=0.04 radius=0.046; visual mesh filename=../meshes/hip.stl scale=1 1 1
- link RL_hip: geometry collision cylinder length=0.04 radius=0.046; visual mesh filename=../meshes/hip.stl scale=1 1 1
- link RR_hip: geometry collision cylinder length=0.04 radius=0.046; visual mesh filename=../meshes/hip.stl scale=1 1 1
- link trunk: geometry collision box size=0.267 0.194 0.114; visual mesh filename=../meshes/trunk.stl scale=1 1 1
Joints:
- removed joint FL_hip_fixed
- removed joint FL_lower_joint
- removed joint FL_toe_fixed
- removed joint FL_upper_joint
- removed joint FR_hip_fixed
- removed joint FR_lower_joint
- removed joint FR_toe_fixed
- removed joint FR_upper_joint
- removed joint RL_hip_fixed
- removed joint RL_lower_joint
- removed joint RL_toe_fixed
- removed joint RL_upper_joint
- removed joint RR_hip_fixed
- removed joint RR_lower_joint
- removed joint RR_toe_fixed
- removed joint RR_upper_joint
- added joint FL_calf_joint: type revolute, parent FL_thigh, child FL_calf, origin xyz=0 0 -0.2 rpy=0 0 0, axis 0 1 0, limit lower=-2.69653369433 upper=-0.916297857297 effort=55 velocity=28.6
- added joint FL_foot_fixed: type fixed, parent FL_calf, child FL_foot, origin xyz=0 0 -0.2 rpy=0 0 0
- added joint FL_thigh_joint: type continuous, parent FL_hip, child FL_thigh, origin xyz=0 0.08505 0 rpy=0 0 0, axis 0 1 0, limit lower=-1.0471975512 upper=4.18879020479 effort=55 velocity=28.6
- added joint FR_calf_joint: type revolute, parent FR_thigh, child FR_calf, origin xyz=0 0 -0.2 rpy=0 0 0, axis 0 1 0, limit lower=-2.69653369433 upper=-0.916297857297 effort=55 velocity=28.6
- added joint FR_foot_fixed: type fixed, parent FR_calf, child FR_foot, origin xyz=0 0 -0.2 rpy=0 0 0
- added joint FR_thigh_joint: type continuous, parent FR_hip, child FR_thigh, origin xyz=0 -0.08505 0 rpy=0 0 0, axis 0 1 0, limit lower=-1.0471975512 upper=4.18879020479 effort=55 velocity=28.6
- added joint RL_calf_joint: type revolute, parent RL_thigh, child RL_calf, origin xyz=0 0 -0.2 rpy=0 0 0, axis 0 1 0, limit lower=-2.69653369433 upper=-0.916297857297 effort=55 velocity=28.6
- added joint RL_foot_fixed: type fixed, parent RL_calf, child RL_foot, origin xyz=0 0 -0.2 rpy=0 0 0
- added joint RL_thigh_joint: type continuous, parent RL_hip, child RL_thigh, origin xyz=0 0.08505 0 rpy=0 0 0, axis 0 1 0, limit lower=-1.0471975512 upper=4.18879020479 effort=55 velocity=28.6
- added joint RR_calf_joint: type revolute, parent RR_thigh, child RR_calf, origin xyz=0 0 -0.2 rpy=0 0 0, axis 0 1 0, limit lower=-2.69653369433 upper=-0.916297857297 effort=55 velocity=28.6
- added joint RR_foot_fixed: type fixed, parent RR_calf, child RR_foot, origin xyz=0 0 -0.2 rpy=0 0 0
- added joint RR_thigh_joint: type continuous, parent RR_hip, child RR_thigh, origin xyz=0 -0.08505 0 rpy=0 0 0, axis 0 1 0, limit lower=-1.0471975512 upper=4.18879020479 effort=55 velocity=28.6
- added joint floating_base: type fixed, parent base, child trunk, origin xyz=0 0 0 rpy=0 0 0

File: unitree_pybullet/unitree_pybullet/data/_aliengo/urdf/aliengo.urdf (robot description, URDF)
Before this commit: robot aliengo_description, 18 links, 17 joints
Links:
- removed link FL_lower
- removed link FL_toe
- removed link FL_upper
- removed link FR_lower
- removed link FR_toe
- removed link FR_upper
- removed link RL_lower
- removed link RL_toe
- removed link RL_upper
- removed link RR_lower
- removed link RR_toe
- removed link RR_upper
- added link FL_calf, mass 0.207; collision box size=0.25 0.0208 0.016; visual mesh filename=../meshes/calf.stl scale=1 1 1
- added link FL_foot, mass 0.06; collision sphere radius=0.0265; visual sphere radius=0.0165
- added link FL_thigh, mass 0.639; collision box size=0.25 0.0374 0.043; visual mesh filename=../meshes/thigh.stl scale=1 1 1
- added link FR_calf, mass 0.207; collision box size=0.25 0.0208 0.016; visual mesh filename=../meshes/calf.stl scale=1 1 1
- added link FR_foot, mass 0.06; collision sphere radius=0.0265; visual sphere radius=0.0165
- added link FR_thigh, mass 0.639; collision box size=0.25 0.0374 0.043; visual mesh filename=../meshes/thigh_mirror.stl scale=1 1 1
- added link RL_calf, mass 0.207; collision box size=0.25 0.0208 0.016; visual mesh filename=../meshes/calf.stl scale=1 1 1
- added link RL_foot, mass 0.06; collision sphere radius=0.0265; visual sphere radius=0.0165
- added link RL_thigh, mass 0.639; collision box size=0.25 0.0374 0.043; visual mesh filename=../meshes/thigh.stl scale=1 1 1
- added link RR_calf, mass 0.207; collision box size=0.25 0.0208 0.016; visual mesh filename=../meshes/calf.stl scale=1 1 1
- added link RR_foot, mass 0.06; collision sphere radius=0.0265; visual sphere radius=0.0165
- added link RR_thigh, mass 0.639; collision box size=0.25 0.0374 0.043; visual mesh filename=../meshes/thigh_mirror.stl scale=1 1 1
- added link base; visual box size=0.001 0.001 0.001
- link FL_hip: geometry collision cylinder length=0.0418 radius=0.046; visual mesh filename=../meshes/hip.stl scale=1 1 1
- link FR_hip: geometry collision cylinder length=0.0418 radius=0.046; visual mesh filename=../meshes/hip.stl scale=1 1 1
- link RL_hip: geometry collision cylinder length=0.0418 radius=0.046; visual mesh filename=../meshes/hip.stl scale=1 1 1
- link RR_hip: geometry collision cylinder length=0.0418 radius=0.046; visual mesh filename=../meshes/hip.stl scale=1 1 1
- link trunk: geometry collision box size=0.647 0.15 0.112; visual mesh filename=../meshes/trunk.stl scale=1 1 1
Joints:
- removed joint FL_lower_joint
- removed joint FL_toe_fixed
- removed joint FL_upper_joint
- removed joint FR_lower_joint
- removed joint FR_toe_fixed
- removed joint FR_upper_joint
- removed joint RL_lower_joint
- removed joint RL_toe_fixed
- removed joint RL_upper_joint
- removed joint RR_lower_joint
- removed joint RR_toe_fixed
- removed joint RR_upper_joint
- added joint FL_calf_joint: type revolute, parent FL_thigh, child FL_calf, origin xyz=0 0 -0.25 rpy=0 0 0, axis 0 1 0, limit lower=-2.77507351067 upper=-0.645771823238 effort=44.4 velocity=40
- added joint FL_foot_fixed: type fixed, parent FL_calf, child FL_foot, origin xyz=0 0 -0.25 rpy=0 0 0
- added joint FL_thigh_joint: type continuous, parent FL_hip, child FL_thigh, origin xyz=0 0.083 0 rpy=0 0 0, axis 0 1 0, limit effort=44.4 velocity=40
- added joint FR_calf_joint: type revolute, parent FR_thigh, child FR_calf, origin xyz=0 0 -0.25 rpy=0 0 0, axis 0 1 0, limit lower=-2.77507351067 upper=-0.645771823238 effort=44.4 velocity=40
- added joint FR_foot_fixed: type fixed, parent FR_calf, child FR_foot, origin xyz=0 0 -0.25 rpy=0 0 0
- added joint FR_thigh_joint: type continuous, parent FR_hip, child FR_thigh, origin xyz=0 -0.083 0 rpy=0 0 0, axis 0 1 0, limit effort=44.4 velocity=40
- added joint RL_calf_joint: type revolute, parent RL_thigh, child RL_calf, origin xyz=0 0 -0.25 rpy=0 0 0, axis 0 1 0, limit lower=-2.77507351067 upper=-0.645771823238 effort=44.4 velocity=40
- added joint RL_foot_fixed: type fixed, parent RL_calf, child RL_foot, origin xyz=0 0 -0.25 rpy=0 0 0
- added joint RL_thigh_joint: type continuous, parent RL_hip, child RL_thigh, origin xyz=0 0.083 0 rpy=0 0 0, axis 0 1 0, limit effort=44.4 velocity=40
- added joint RR_calf_joint: type revolute, parent RR_thigh, child RR_calf, origin xyz=0 0 -0.25 rpy=0 0 0, axis 0 1 0, limit lower=-2.77507351067 upper=-0.645771823238 effort=44.4 velocity=40
- added joint RR_foot_fixed: type fixed, parent RR_calf, child RR_foot, origin xyz=0 0 -0.25 rpy=0 0 0
- added joint RR_thigh_joint: type continuous, parent RR_hip, child RR_thigh, origin xyz=0 -0.083 0 rpy=0 0 0, axis 0 1 0, limit effort=44.4 velocity=40
- added joint floating_base: type fixed, parent base, child trunk, origin xyz=0 0 0 rpy=0 0 0

File: unitree_pybullet/unitree_pybullet/data/laikago/urdf/laikago.urdf (robot description, URDF)
Before this commit: robot laikago_description, 13 links, 12 joints
Links:
- removed link FL_calf
- removed link FL_hip
- removed link FL_thigh
- removed link FR_calf
- removed link FR_hip
- removed link FR_thigh
- removed link RL_calf
- removed link RL_hip
- removed link RL_thigh
- removed link RR_calf
- removed link RR_hip
- removed link RR_thigh
- removed link trunk
- added link FL_hip_motor, mass 1.095; collision mesh filename=../meshes/hip_motor.stl scale=1 1 1; visual mesh filename=../meshes/hip_motor.obj scale=1 1 1
- added link FL_lower_leg, mass 0.241; collision mesh filename=../meshes/lower_leg_3_collision.stl scale=1 1 1; visual mesh filename=../meshes/lower_leg3.obj scale=1 1 1
- added link FL_upper_leg, mass 1.527; collision mesh filename=../meshes/upper_leg_left_vhacd.obj scale=1 1 1; visual mesh filename=../meshes/upper_leg_left.obj scale=1 1 1
- added link FR_hip_motor, mass 1.095; collision mesh filename=../meshes/hip_motor_mirror.stl scale=1 1 1; visual mesh filename=../meshes/hip_motor_mirror.obj scale=1 1 1
- added link FR_lower_leg, mass 0.241; collision mesh filename=../meshes/lower_leg_3_collision.stl scale=1 1 1; visual mesh filename=../meshes/lower_leg3.obj scale=1 1 1
- added link FR_upper_leg, mass 1.527; collision mesh filename=../meshes/upper_leg_right_vhacd.obj scale=1 1 1; visual mesh filename=../meshes/upper_leg_mirror.obj scale=1 1 1
- added link RL_hip_motor, mass 1.095; collision mesh filename=../meshes/hip_motor.stl scale=1 1 1; visual mesh filename=../meshes/hip_motor.obj scale=1 1 1
- added link RL_lower_leg, mass 0.241; collision mesh filename=../meshes/lower_leg_3_collision.stl scale=1 1 1; visual mesh filename=../meshes/lower_leg3.obj scale=1 1 1
- added link RL_upper_leg, mass 1.527; collision mesh filename=../meshes/upper_leg_left_vhacd.obj scale=1 1 1; visual mesh filename=../meshes/upper_leg_left2.obj scale=1 1 1
- added link RR_hip_motor, mass 1.095; collision mesh filename=../meshes/hip_motor_mirror.stl scale=1 1 1; visual mesh filename=../meshes/hip_motor_mirror.obj scale=1 1 1
- added link RR_lower_leg, mass 0.241; collision mesh filename=../meshes/lower_leg_3_collision.stl scale=1 1 1; visual mesh filename=../meshes/lower_leg3.obj scale=1 1 1
- added link RR_upper_leg, mass 1.527; collision mesh filename=../meshes/upper_leg_right_vhacd.obj scale=1 1 1; visual mesh filename=../meshes/upper_leg_mirror2.obj scale=1 1 1
- added link chassis, mass 13.715; collision mesh filename=../meshes/chassis_vhacd_mod.obj scale=1 1 1; visual mesh filename=../meshes/chassis.obj scale=1 1 1
Joints:
- removed joint FL_calf_joint
- removed joint FL_hip_joint
- removed joint FL_thigh_joint
- removed joint FR_calf_joint
- removed joint FR_hip_joint
- removed joint FR_thigh_joint
- removed joint RL_calf_joint
- removed joint RL_hip_joint
- removed joint RL_thigh_joint
- removed joint RR_calf_joint
- removed joint RR_hip_joint
- removed joint RR_thigh_joint
- added joint FL_hip_motor_2_chassis_joint: type continuous, parent chassis, child FL_hip_motor, origin xyz=0.0817145 0 0.242889 rpy=0 0 0, axis 0 0 1, limit effort=100 velocity=100
- added joint FL_lower_leg_2_upper_leg_joint: type continuous, parent FL_upper_leg, child FL_lower_leg, origin xyz=-0.02069  -0.20833  -0.1422 rpy=0 0 0, axis 1 0 0, limit effort=100 velocity=100
- added joint FL_upper_leg_2_hip_motor_joint: type continuous, parent FL_hip_motor, child FL_upper_leg, origin xyz=0.055855  0 0 rpy=0 0 0, axis 1 0 0, limit effort=100 velocity=100
- added joint FR_hip_motor_2_chassis_joint: type continuous, parent chassis, child FR_hip_motor, origin xyz=-0.0817145 0 0.242889 rpy=0 0 0, axis 0 0 -1, limit effort=100 velocity=100
- added joint FR_lower_leg_2_upper_leg_joint: type continuous, parent FR_upper_leg, child FR_lower_leg, origin xyz=0.02069  -0.20833  -0.1422 rpy=0 0 0, axis 1 0 0, limit effort=100 velocity=100
- added joint FR_upper_leg_2_hip_motor_joint: type continuous, parent FR_hip_motor, child FR_upper_leg, origin xyz=-0.053565 0 0 rpy=0 0 0, axis 1 0 0, limit effort=100 velocity=100
- added joint RL_hip_motor_2_chassis_joint: type continuous, parent chassis, child RL_hip_motor, origin xyz=0.0817145 0 -0.194401 rpy=0 0 0, axis 0 0 1, limit effort=100 velocity=100
- added joint RL_lower_leg_2_upper_leg_joint: type continuous, parent RL_upper_leg, child RL_lower_leg, origin xyz=-0.02069  -0.20833  -0.1422 rpy=0 0 0, axis 1 0 0, limit effort=100 velocity=100
- added joint RL_upper_leg_2_hip_motor_joint: type continuous, parent RL_hip_motor, child RL_upper_leg, origin xyz=0.055855  0 0 rpy=0 0 0, axis 1 0 0, limit effort=100 velocity=100
- added joint RR_hip_motor_2_chassis_joint: type continuous, parent chassis, child RR_hip_motor, origin xyz=-0.0817145 0 -0.194401 rpy=0 0 0, axis 0 0 -1, limit effort=100 velocity=100
- added joint RR_lower_leg_2_upper_leg_joint: type continuous, parent RR_upper_leg, child RR_lower_leg, origin xyz=0.02069  -0.20833  -0.1422 rpy=0 0 0, axis 1 0 0, limit effort=100 velocity=100
- added joint RR_upper_leg_2_hip_motor_joint: type continuous, parent RR_hip_motor, child RR_upper_leg, origin xyz=-0.053565 0 0 rpy=0 0 0, axis 1 0 0, limit effort=100 velocity=100
